File: hardware/CAN transreciver.sch (KiCad schematic (older format))
At the start: 10 parts, among them U3 ATA6561-GAQW-N

Commit message: Updated to be compatible with KiCad 6.0.0, changed chematics layouts to fit in A4 worksheet and finished routing the rest of the signals.
Parts:
- removed U3: ATA6561-GAQW-N, Package_DFN_QFN:DFN-8-1EP_3x3mm_P0.65mm_EP1.55x2.4mm, symbol Interface_CAN_LIN:MCP2562-E-MF
- added U11: MCP2558FD-xSN, Package_SO:SOIC-8_3.9x4.9mm_P1.27mm, symbol Interface_CAN_LIN:MCP2558FD-xSN
Connections:
- net +3V3_VIO: now also U11.5 (VIO)
- net +5V_CAN_VDD: now also U11.3 (VDD)
- net CAN-RX: now also U11.4 (RXD)
- net CAN-TX: now also U11.1 (TXD)
- net CANH: now also U11.7 (CANH)
- net CANL: now also U11.6 (CANL)
- net GND: now also U11.2 (VSS)
- net SHDN: now also U11.8 (S)
Changed lines of the file:
@@
 $Descr A4 11693 8268
 encoding utf-8
-Sheet 8 20
+Sheet 2 24
 Title "High-Speed CAN Transceiver"
 Date ""
@@
 Comment4 ""
 $EndDescr
-$Comp
-L Interface_CAN_LIN:MCP2562-E-MF U3
-U 1 1 61A168ED
-P 5700 3950
-AR Path="/61A14ADD/61A168ED" Ref="U3"  Part="1"
-AR Path="/61A9D384/61A168ED" Ref="U4"  Part="1"
-AR Path="/61A5C8B4/61A168ED" Ref="U11"  Part="1"
-F 0 "U11" H 6100 4450 50  0000 C CNN
-F 1 "ATA6561-GAQW-N" H 6200 4350 50  0000 C CNN
-F 2 "Package_DFN_QFN:DFN-8-1EP_3x3mm_P0.65mm_EP1.55x2.4mm" H 5700 3450 50  0001 C CIN
-F 3 "https://pl.mouser.com/datasheet/2/268/ATA6560_ATA6561_High_Speed_CAN_Transceiver_DS20005-1384933.pdf" H 5700 3950 50  0001 C CNN
-	1    5700 3950
-	1    0    0    -1
-$EndComp
 $Comp
 L power:GND #PWR015
@@
 	1    0    0    -1
 $EndComp
-Wire Wire Line
-	5700 4450 5700 4400
-Wire Wire Line
-	5700 4400 5600 4400
-Wire Wire Line
-	5600 4400 5600 4350
-Wire Wire Line
-	5700 4400 5700 4350
-Connection ~ 5700 4400
 Wire Wire Line
 	6200 3850 6700 3850
@@
 	1    0    0    -1
 $EndComp
+$Comp
+L Interface_CAN_LIN:MCP2558FD-xSN U11
+U 1 1 63ED2897
+P 5700 3950
+F 0 "U11" H 5700 4531 50  0000 C CNN
+F 1 "MCP2558FD-xSN" H 5700 4440 50  0000 C CNN
+F 2 "Package_SO:SOIC-8_3.9x4.9mm_P1.27mm" H 5700 3350 50  0001 C CNN
+F 3 "https://ww1.microchip.com/downloads/en/DeviceDoc/20005533A.pdf" H 5700 3950 50  0001 C CNN
+	1    5700 3950
+	1    0    0    -1
+$EndComp
+Wire Wire Line
+	5700 4350 5700 4450
 $EndSCHEMATC
