File: hardware/Digital_Output.sch (KiCad schematic (older format))
At the start: 4 parts, among them U16 MCP14A0052T

Commit message: 1. added 2X20 connector, \n 2. changed the footprints of schootkies and zenner diodes to a bigger ones, \n 3. changed pcb layout entirely couse duck me, that connector i too duking BIG.
Parts:
- U16: symbol MCP14A0052T:MCP14A0052T -> SB-Spoko-Bezpieczniki-rescue:MCP14A0052T-MCP14A0052T
Changed lines of the file:
@@
 $Descr A4 11693 8268
 encoding utf-8
-Sheet 14 20
+Sheet 13 20
 Title ""
 Date ""
@@
 AR Path="/61E9FD3E/61A9FB37" Ref="#PWR0120"  Part="1"
 AR Path="/61ECEEF9/61A9FB37" Ref="#PWR0116"  Part="1"
-F 0 "#PWR0116" H 4800 3700 50  0001 C CNN
+F 0 "#PWR0120" H 4800 3700 50  0001 C CNN
 F 1 "+5V" H 4815 4023 50  0000 C CNN
 F 2 "" H 4800 3850 50  0001 C CNN
@@
 AR Path="/61E9FD3E/61A9FD58" Ref="#PWR0121"  Part="1"
 AR Path="/61ECEEF9/61A9FD58" Ref="#PWR0117"  Part="1"
-F 0 "#PWR0117" H 4800 4600 50  0001 C CNN
+F 0 "#PWR0121" H 4800 4600 50  0001 C CNN
 F 1 "GND" H 4805 4677 50  0000 C CNN
 F 2 "" H 4800 4850 50  0001 C CNN
@@
 AR Path="/61E9FD3E/61AA37F7" Ref="D25"  Part="1"
 AR Path="/61ECEEF9/61AA37F7" Ref="D24"  Part="1"
-F 0 "D24" V 4239 4632 50  0000 R CNN
+F 0 "D23" V 4239 4632 50  0000 R CNN
 F 1 "LED_GREEN" V 4148 4632 50  0000 R CNN
 F 2 "Diode_SMD:D_0603_1608Metric" H 4200 4750 50  0001 C CNN
@@
 AR Path="/61E9FD3E/61AA3B2C" Ref="R45"  Part="1"
 AR Path="/61ECEEF9/61AA3B2C" Ref="R43"  Part="1"
-F 0 "R43" H 4270 5196 50  0000 L CNN
+F 0 "R41" H 4270 5196 50  0000 L CNN
 F 1 "1k" H 4270 5105 50  0000 L CNN
 F 2 "Resistor_SMD:R_0603_1608Metric" V 4130 5150 50  0001 C CNN
@@
 AR Path="/61E9FD3E/61AA3C66" Ref="#PWR0122"  Part="1"
 AR Path="/61ECEEF9/61AA3C66" Ref="#PWR0118"  Part="1"
-F 0 "#PWR0118" H 4200 5100 50  0001 C CNN
+F 0 "#PWR0122" H 4200 5100 50  0001 C CNN
 F 1 "GND" H 4205 5177 50  0000 C CNN
 F 2 "" H 4200 5350 50  0001 C CNN
@@
 AR Path="/61E9FD3E/61AA4F82" Ref="C40"  Part="1"
 AR Path="/61ECEEF9/61AA4F82" Ref="C39"  Part="1"
-F 0 "C39" V 4821 4100 50  0000 C CNN
+F 0 "C38" V 4821 4100 50  0000 C CNN
 F 1 "100nF" V 4912 4100 50  0000 C CNN
 F 2 "Capacitor_SMD:C_0603_1608Metric" H 5050 4100 50  0001 C CNN
@@
 AR Path="/61E9FD3E/61AA6A32" Ref="#PWR0123"  Part="1"
 AR Path="/61ECEEF9/61AA6A32" Ref="#PWR0119"  Part="1"
-F 0 "#PWR0119" H 5200 3850 50  0001 C CNN
+F 0 "#PWR0123" H 5200 3850 50  0001 C CNN
 F 1 "GND" V 5205 3972 50  0000 R CNN
 F 2 "" H 5200 4100 50  0001 C CNN
@@
 100R
 $Comp
-L MCP14A0052T:MCP14A0052T U16
+L SB-Spoko-Bezpieczniki-rescue:MCP14A0052T-MCP14A0052T U16
 U 1 1 61E992D7
 P 4800 4450
@@
 AR Path="/61E9FD3E/61E992D7" Ref="U18"  Part="1"
 AR Path="/61ECEEF9/61E992D7" Ref="U17"  Part="1"
-F 0 "U17" H 5244 4496 50  0000 L CNN
+AR Path="/61E992D7" Ref="U17"  Part="1"
+F 0 "U16" H 5244 4496 50  0000 L CNN
 F 1 "MCP14A0052T" H 5244 4405 50  0000 L CNN
 F 2 "Package_TO_SOT_SMD:SOT-23-6" H 4800 3850 50  0001 C CIN

Commit message: Updated to be compatible with KiCad 6.0.0, changed chematics layouts to fit in A4 worksheet and finished routing the rest of the signals.
Changed lines of the file:
@@
 $Descr A4 11693 8268
 encoding utf-8
-Sheet 13 20
+Sheet 7 24
 Title ""
 Date ""
@@
 AR Path="/61E9FD3E/61AA37F7" Ref="D25"  Part="1"
 AR Path="/61ECEEF9/61AA37F7" Ref="D24"  Part="1"
-F 0 "D23" V 4239 4632 50  0000 R CNN
+F 0 "D25" V 4239 4632 50  0000 R CNN
 F 1 "LED_GREEN" V 4148 4632 50  0000 R CNN
 F 2 "Diode_SMD:D_0603_1608Metric" H 4200 4750 50  0001 C CNN
@@
 AR Path="/61E9FD3E/61AA3B2C" Ref="R45"  Part="1"
 AR Path="/61ECEEF9/61AA3B2C" Ref="R43"  Part="1"
-F 0 "R41" H 4270 5196 50  0000 L CNN
+F 0 "R45" H 4270 5196 50  0000 L CNN
 F 1 "1k" H 4270 5105 50  0000 L CNN
 F 2 "Resistor_SMD:R_0603_1608Metric" V 4130 5150 50  0001 C CNN
@@
 AR Path="/61E9FD3E/61AA4F82" Ref="C40"  Part="1"
 AR Path="/61ECEEF9/61AA4F82" Ref="C39"  Part="1"
-F 0 "C38" V 4821 4100 50  0000 C CNN
+F 0 "C40" V 4821 4100 50  0000 C CNN
 F 1 "100nF" V 4912 4100 50  0000 C CNN
 F 2 "Capacitor_SMD:C_0603_1608Metric" H 5050 4100 50  0001 C CNN
@@
 AR Path="/61ECEEF9/61E992D7" Ref="U17"  Part="1"
 AR Path="/61E992D7" Ref="U17"  Part="1"
-F 0 "U16" H 5244 4496 50  0000 L CNN
+F 0 "U18" H 5244 4496 50  0000 L CNN
 F 1 "MCP14A0052T" H 5244 4405 50  0000 L CNN
 F 2 "Package_TO_SOT_SMD:SOT-23-6" H 4800 3850 50  0001 C CIN
