File: hardware/SB-Spoko Bezpieczniki.sch (KiCad schematic (older format))
At the start: 62 parts, among them IC1 STM32L4P5RET6, J1 SWD, SW1 RESET, U1 AS222-35PN-933, U2 LM2596S-12, U3 LM2596S-5, U4 LP2950-3.3_TO92, Y1 THE_CLOCK

Commit message: 1. added 2X20 connector, \n 2. changed the footprints of schootkies and zenner diodes to a bigger ones, \n 3. changed pcb layout entirely couse duck me, that connector i too duking BIG.
Parts:
- added J2: Conn_02x20_Odd_Even, Connector_IDC:IDC-Header_2x20-1MP_P2.54mm_Latch_Horizontal, symbol Connector_Generic:Conn_02x20_Odd_Even
- D3, D4, D5, D6, D7, D8: footprint Diode_SMD:D_0603_1608Metric -> Diode_SMD:D_SMA
Connections:
- net labels added: CAR_CAN+, CAR_CAN-, INV_CAN+, INV_CAN-
- wire segments 421 -> 463
- no-connect marks 67 -> 65
Changed lines of the file:
@@
 N_TD
 $Sheet
-S 19350 14000 750  300
+S 19250 14000 750  300
 U 61A5C8B4
 F0 "CAN transreciver" 50
 F1 "CAN transreciver.sch" 50
-F2 "CAN-RX" O L 19350 14100 50
-F3 "CAN-TX" I L 19350 14200 50
-F4 "CANH" B R 20100 14100 50
-F5 "CANL" B R 20100 14200 50
+F2 "CAN-RX" O L 19250 14100 50
+F3 "CAN-TX" I L 19250 14200 50
+F4 "CANH" B R 20000 14100 50
+F5 "CANL" B R 20000 14200 50
 $EndSheet
 $Sheet
@@
 $EndSheet
 Wire Wire Line
-	18950 14100 19350 14100
-Text Label 18950 14100 0    50   ~ 0
+	18850 14100 19250 14100
+Text Label 18850 14100 0    50   ~ 0
 CAN_RX
-Text Label 18950 14200 0    50   ~ 0
+Text Label 18850 14200 0    50   ~ 0
 CAN_TX
 Wire Wire Line
-	19350 14200 18950 14200
-Wire Wire Line
-	20450 14100 20100 14100
-Wire Wire Line
-	20450 14200 20100 14200
-Text Label 20450 14100 2    50   ~ 0
-CAN_L
-Text Label 20450 14200 2    50   ~ 0
-CAN_H
+	19250 14200 18850 14200
 Wire Wire Line
 	9950 4500 9950 4400
@@
 $EndComp
 Wire Wire Line
-	11500 6950 10750 6950
-Wire Wire Line
-	11500 6750 10750 6750
-Text Label 11500 6950 2    50   ~ 0
-STM_SOFT_ERROR
-Text Label 11500 6750 2    50   ~ 0
-STM_???
-Text Label 11500 7050 2    50   ~ 0
-STM_OK
-Wire Wire Line
-	11500 7050 10750 7050
-Wire Wire Line
 	1450 1600 1350 1600
 Wire Wire Line
@@
 Wire Notes Line width 20 rgb(132, 0, 0)
 	14050 2900 14050 16050
-Text Notes 17500 12800 2    787  ~ 157
+Text Notes 17550 10050 2    787  ~ 157
 BUS
-Text Notes 17450 11750 0    39   ~ 8
+Text Notes 17500 9000 0    39   ~ 8
 TM
 Wire Notes Line width 20 rgb(132, 0, 0)
 	18650 7150 22900 7150
-Text Notes 14950 13150 0    50   ~ 0
+Text Notes 15000 10400 0    50   ~ 0
 miejsce na przyszłą taśme/magistrale komunikacyją z resztą boxa\n
-Wire Wire Line
-	1350 9500 2100 9500
-Wire Wire Line
-	1350 9400 2100 9400
-Text Label 1350 9500 0    50   ~ 0
-CAN_L
-Text Label 1350 9400 0    50   ~ 0
-CAN_H
 Text Notes 21250 4800 0    50   ~ 0
 gdzie?\n
@@
 L power:+5V #PWR0103
 U 1 1 62E35228
-P 15450 13800
-F 0 "#PWR0103" H 15450 13650 50  0001 C CNN
-F 1 "+5V" V 15465 13928 50  0000 L CNN
-F 2 "" H 15450 13800 50  0001 C CNN
-F 3 "" H 15450 13800 50  0001 C CNN
-	1    15450 13800
+P 15750 14950
+F 0 "#PWR0103" H 15750 14800 50  0001 C CNN
+F 1 "+5V" V 15765 15078 50  0000 L CNN
+F 2 "" H 15750 14950 50  0001 C CNN
+F 3 "" H 15750 14950 50  0001 C CNN
+	1    15750 14950
 	1    0    0    -1
 $EndComp
@@
 L power:GND #PWR0104
 U 1 1 62E6D9BC
-P 15650 13700
-F 0 "#PWR0104" H 15650 13450 50  0001 C CNN
-F 1 "GND" H 15655 13527 50  0000 C CNN
-F 2 "" H 15650 13700 50  0001 C CNN
-F 3 "" H 15650 13700 50  0001 C CNN
-	1    15650 13700
+P 15950 14850
+F 0 "#PWR0104" H 15950 14600 50  0001 C CNN
+F 1 "GND" H 15955 14677 50  0000 C CNN
+F 2 "" H 15950 14850 50  0001 C CNN
+F 3 "" H 15950 14850 50  0001 C CNN
+	1    15950 14850
 	1    0    0    -1
 $EndComp
 Wire Wire Line
-	15950 13450 15950 13800
+	16250 14600 16250 14950
 Wire Wire Line
-	16250 13450 16250 13800
-Text Label 15950 13450 3    50   ~ 0
+	16550 14600 16550 14950
+Text Label 16250 14600 3    50   ~ 0
 CAN_L
-Text Label 16250 13450 3    50   ~ 0
+Text Label 16550 14600 3    50   ~ 0
 CAN_H
 Wire Wire Line
-	16500 13450 16500 14300
-Text Label 16500 13450 3    50   ~ 0
+	16800 14600 16800 15450
+Text Label 16800 14600 3    50   ~ 0
 RTDS_GATE
 Wire Wire Line
-	16750 13450 16750 14300
-Text Label 16750 13450 3    50   ~ 0
+	17050 14600 17050 15450
+Text Label 17050 14600 3    50   ~ 0
 BREAK_LIGHT_GATE
 $Comp
@@
 NoConn ~ 2100 9000
 NoConn ~ 2100 8500
-NoConn ~ 2100 8400
-NoConn ~ 2100 8300
 NoConn ~ 2100 8100
 NoConn ~ 2100 8000
@@
 NoConn ~ 2500 6800
 NoConn ~ 2500 6700
-NoConn ~ 2500 6600
-NoConn ~ 2500 6500
 NoConn ~ 2500 6400
 NoConn ~ 2500 6300
@@
 F 0 "D7" V 8350 12300 50  0000 C CNN
 F 1 "D_SCH" V 8450 12300 50  0001 C CNN
-F 2 "Diode_SMD:D_0603_1608Metric" V 8400 12200 50  0001 C CNN
+F 2 "Diode_SMD:D_SMA" V 8400 12200 50  0001 C CNN
 F 3 "~" V 8400 12200 50  0001 C CNN
 	1    8400 12200
@@
 F 0 "D5" V 6000 12350 50  0000 C CNN
 F 1 "D_SCH" V 6100 12350 50  0001 C CNN
-F 2 "Diode_SMD:D_0603_1608Metric" V 6050 12250 50  0001 C CNN
+F 2 "Diode_SMD:D_SMA" V 6050 12250 50  0001 C CNN
 F 3 "~" V 6050 12250 50  0001 C CNN
 	1    6050 12250
@@
 F 0 "D3" V 5750 12400 50  0000 R CNN
 F 1 "D_ZEN" V 5850 12350 50  0001 R CNN
-F 2 "Diode_SMD:D_0603_1608Metric" V 5800 12250 50  0001 C CNN
+F 2 "Diode_SMD:D_SMA" V 5800 12250 50  0001 C CNN
 F 3 "~" V 5800 12250 50  0001 C CNN
 	1    5800 12250
@@
 F 0 "D8" V 8400 15050 50  0000 C CNN
 F 1 "D_SCH" V 8500 15050 50  0001 C CNN
-F 2 "Diode_SMD:D_0603_1608Metric" V 8450 14950 50  0001 C CNN
+F 2 "Diode_SMD:D_SMA" V 8450 14950 50  0001 C CNN
 F 3 "~" V 8450 14950 50  0001 C CNN
 	1    8450 14950
@@
 F 0 "D6" V 6050 15050 50  0000 C CNN
 F 1 "D_SCH" V 6150 15050 50  0001 C CNN
-F 2 "Diode_SMD:D_0603_1608Metric" V 6100 14950 50  0001 C CNN
+F 2 "Diode_SMD:D_SMA" V 6100 14950 50  0001 C CNN
 F 3 "~" V 6100 14950 50  0001 C CNN
 	1    6100 14950
@@
 F 0 "D4" V 5800 15100 50  0000 R CNN
 F 1 "D_ZEN" V 5900 15050 50  0001 R CNN
-F 2 "Diode_SMD:D_0603_1608Metric" V 5850 14950 50  0001 C CNN
+F 2 "Diode_SMD:D_SMA" V 5850 14950 50  0001 C CNN
 F 3 "~" V 5850 14950 50  0001 C CNN
 	1    5850 14950
@@
 $EndComp
 Wire Wire Line
-	11500 6850 10750 6850
-Text Label 11500 6850 2    50   ~ 0
-STM_FATAL_ERROR
-Wire Wire Line
-	3250 7900 2500 7900
-Text Label 3250 7900 2    50   ~ 0
-HVD
-Wire Wire Line
-	3250 8000 2500 8000
-Text Label 3250 8000 2    50   ~ 0
-TSMS
-Wire Wire Line
-	2500 8700 3250 8700
-Text Label 3250 8700 2    50   ~ 0
-TD
-Wire Wire Line
-	2500 8800 3250 8800
+	3250 8800 2500 8800
 Text Label 3250 8800 2    50   ~ 0
-SPARE
-Wire Wire Line
-	3250 8900 2500 8900
-Text Label 3250 8900 2    50   ~ 0
-AMS
+HVD
 $Comp
 L Autosport:AS222-35PN-933 U1
@@
 	1    0    0    -1
 $EndComp
+$Comp
+L Connector_Generic:Conn_02x20_Odd_Even J2
+U 1 1 61BF6F6C
+P 16400 12600
+F 0 "J2" H 16450 11375 50  0000 C CNN
+F 1 "Conn_02x20_Odd_Even" H 16450 11466 50  0000 C CNN
+F 2 "Connector_IDC:IDC-Header_2x20-1MP_P2.54mm_Latch_Horizontal" H 16400 12600 50  0001 C CNN
+F 3 "~" H 16400 12600 50  0001 C CNN
+	1    16400 12600
+	-1   0    0    1
+$EndComp
+Wire Wire Line
+	16100 13500 16000 13500
+Wire Wire Line
+	16100 13400 16000 13400
+Wire Wire Line
+	16100 13300 16000 13300
+Wire Wire Line
+	16100 13200 16000 13200
+Wire Wire Line
+	16100 13100 16000 13100
+Wire Wire Line
+	16100 13000 16000 13000
+Wire Wire Line
+	16100 12900 16000 12900
+Wire Wire Line
+	16100 12800 16000 12800
+Wire Wire Line
+	16100 12700 16000 12700
+Wire Wire Line
+	16100 12600 16000 12600
+Wire Wire Line
+	16100 12500 16000 12500
+Wire Wire Line
+	16100 12400 16000 12400
+Wire Wire Line
+	16100 12300 16000 12300
+Wire Wire Line
+	16100 12200 16000 12200
+Wire Wire Line
+	16100 12100 16000 12100
+Wire Wire Line
+	16100 12000 16000 12000
+Wire Wire Line
+	16100 11900 16000 11900
+Wire Wire Line
+	16100 11800 16000 11800
+Wire Wire Line
+	16100 11700 16000 11700
+Wire Wire Line
+	16100 11600 16000 11600
+Wire Wire Line
+	16700 13500 16600 13500
+Wire Wire Line
+	16700 13400 16600 13400
+Wire Wire Line
+	16700 13300 16600 13300
+Wire Wire Line
+	16700 13200 16600 13200
+Wire Wire Line
+	16700 13100 16600 13100
+Wire Wire Line
+	16700 13000 16600 13000
+Wire Wire Line
+	16700 12900 16600 12900
+Wire Wire Line
+	16700 12800 16600 12800
+Wire Wire Line
+	16700 12700 16600 12700
+Wire Wire Line
+	16700 12600 16600 12600
+Wire Wire Line
+	16700 12500 16600 12500
+Wire Wire Line
+	16700 12400 16600 12400
+Wire Wire Line
+	16700 12300 16600 12300
+Wire Wire Line
+	16700 12200 16600 12200
+Wire Wire Line
+	16700 12100 16600 12100
+Wire Wire Line
+	16700 12000 16600 12000
+Wire Wire Line
+	16700 11900 16600 11900
+Wire Wire Line
+	16700 11800 16600 11800
+Wire Wire Line
+	16700 11700 16600 11700
+Wire Wire Line
+	16700 11600 16600 11600
+Wire Wire Line
+	2500 8000 3250 8000
+Text Label 3250 8000 2    50   ~ 0
+SPARE
+Wire Wire Line
+	2500 8900 3250 8900
+Text Label 3250 8900 2    50   ~ 0
+TD
+Text Label 3250 7900 2    50   ~ 0
+TSMS
+Wire Wire Line
+	3250 7900 2500 7900
+Text Label 3250 8700 2    50   ~ 0
+AMS
+Wire Wire Line
+	3250 8700 2500 8700
+Wire Wire Line
+	1350 8400 2100 8400
+Wire Wire Line
+	1350 8300 2100 8300
+Text Label 1350 8400 0    50   ~ 0
+INV_CAN-
+Text Label 1350 8300 0    50   ~ 0
+INV_CAN+
+Wire Wire Line
+	20550 14100 20000 14100
+Wire Wire Line
+	20550 14200 20000 14200
+Text Label 20550 14100 2    50   ~ 0
+CAR_CAN-
+Text Label 20550 14200 2    50   ~ 0
+CAR_CAN+
+NoConn ~ 2500 6500
+NoConn ~ 2500 6600
+Text Label 1350 9400 0    50   ~ 0
+CAR_CAN+
+Text Label 1350 9500 0    50   ~ 0
+CAR_CAN-
+Wire Wire Line
+	1350 9400 2100 9400
+Wire Wire Line
+	1350 9500 2100 9500
+Wire Notes Line rgb(0, 194, 194)
+	1525 13440 1645 13420
+Wire Notes Line rgb(0, 194, 194)
+	1645 13420 1645 13745
+Wire Notes Line rgb(0, 194, 194)
+	1645 13745 1525 13745
+Wire Notes Line rgb(0, 194, 194)
+	1525 13745 1525 13440
+Text Label 11500 6950 2    50   ~ 0
+STM_FATAL_ERROR
+Wire Wire Line
+	11500 6950 10750 6950
+Wire Wire Line
+	11500 6750 10750 6750
+Text Label 11500 6750 2    50   ~ 0
+STM_OK
+Text Label 11500 7050 2    50   ~ 0
+STM_???
+Text Label 11500 6850 2    50   ~ 0
+STM_SOFT_ERROR
+Wire Wire Line
+	11500 7050 10750 7050
+Wire Wire Line
+	11500 6850 10750 6850
 $EndSCHEMATC

Commit message: Updated to be compatible with KiCad 6.0.0, changed chematics layouts to fit in A4 worksheet and finished routing the rest of the signals.
Connections:
- net labels added: MONO_NTC, RES_COS+, RES_COS-, RES_REF+, RES_REF-, RES_SIN+, RES_SIN-, SP_L+, SP_L-, USB_DEBUG_DM, USB_DEBUG_DP, USB_DM, USB_DP, V_SAFETY, WATER_NTC_1, WATER_NTC_2, WATER_P, WSS_FL, WSS_FR, WSS_RL, WSS_RR
- net labels removed: CAN_H, CAN_L, SAFETY
- wire segments 463 -> 529
- no-connect marks 65 -> 56
Other:
- note removed: "Narazie rokład power tak zostawiłem"
- note removed: "miejsce na przyszłą taśme/magistrale komunikacyją z resztą boxa\n"
