File: hardware/_autosave-Connectors.sch (KiCad schematic (older format))
At the start: 63 parts, among them IC1 STM32L4P5RET6, J1 SWD, J2 Conn_02x20_Odd_Even, SW1 RESET, U1 AS222-35PN-933, U2 LM2596S-12, U3 LM2596S-5, U4 LP2950-3.3_TO92, Y1 THE_CLOCK

Commit message: Updated to be compatible with KiCad 6.0.0, changed chematics layouts to fit in A4 worksheet and finished routing the rest of the signals.
Parts:
- removed C10, C11, C12, C13, C14, C2, C3, C33, C37, C41, C6, C7: 100nF, Capacitor_SMD:C_0603_1608Metric, symbol Device:C_Small
- removed C34, C35: 22pF, Capacitor_SMD:C_0603_1608Metric, symbol Device:C_Small
- removed C36, C4, C5, C8, C9: 10pF, Capacitor_SMD:CP_Elec_6.3x7.7, symbol Device:CP_Small
- removed D1, D2: IN, Diode_SMD:D_0603_1608Metric, symbol Device:LED_Small
- removed D10, D11, D9: OUT, Diode_SMD:D_0603_1608Metric, symbol Device:LED_Small
- removed D19: I'M FINE, Diode_SMD:D_0603_1608Metric, symbol Device:LED_Small
- removed D20: I_AM_ON_FIRE!!!, Diode_SMD:D_0603_1608Metric, symbol Device:LED_Small
- removed D21: COULD_BE_BETTER, Diode_SMD:D_0603_1608Metric, symbol Device:LED_Small
- removed D22: WHAT_THE_F?, Diode_SMD:D_0603_1608Metric, symbol Device:LED_Small
- removed D3, D4: D_ZEN, Diode_SMD:D_SMA, symbol Device:D_Zener_Small
- removed D5, D6, D7, D8: D_SCH, Diode_SMD:D_SMA, symbol Device:D_Schottky_Small
- removed F1, F2, F4: Polyfuse, Fuse:Fuse_2010_5025Metric, symbol Device:Polyfuse
- removed FB3: FB, Inductor_SMD:L_0603_1608Metric, symbol Device:Ferrite_Bead_Small
- removed IC1: STM32L4P5RET6, STM32L4P5RET6:QFP50P1200X1200X160-64N, symbol STM32L4P5RET6:STM32L4P5RET6
- removed J1: SWD, Connector_PinHeader_2.54mm:PinHeader_1x06_P2.54mm_Vertical, symbol Connector:Conn_01x06_Male
- removed L1, L2, L3, L4: 22uH, Inductor_SMD:L_12x12mm_H8mm, symbol Device:L_Small
- removed R1, R2, R20, R4, R5, R6: 1k, Resistor_SMD:R_0603_1608Metric, symbol Device:R
- removed R24: 100k, Resistor_SMD:R_0603_1608Metric, symbol Device:R_Small
- removed R3: 10k, Resistor_SMD:R_0603_1608Metric, symbol Device:R_Small
- removed R37, R38, R39, R40: 470, Resistor_SMD:R_0603_1608Metric, symbol Device:R
- removed SW1: RESET, Button_Switch_THT:SW_PUSH_6mm, symbol Switch:SW_Push
- removed U2: LM2596S-12, Package_TO_SOT_SMD:TO-263-5_TabPin3, symbol Regulator_Switching:LM2596S-ADJ
- removed U3: LM2596S-5, Package_TO_SOT_SMD:TO-263-5_TabPin3, symbol Regulator_Switching:LM2596S-5
- removed U4: LP2950-3.3_TO92, Package_TO_SOT_SMD:SOT-223-3_TabPin2, symbol Regulator_Linear:LP2950-3.3_TO92
- removed Y1: THE_CLOCK, Crystal:Crystal_SMD_HC49-SD, symbol Device:Crystal_Small
Connections:
- no-connect marks 56 -> 24
Other:
- note removed: "12V Converter\n"
- note removed: "3.3V Inline converter\n"
- note removed: "5V Converter\n"
- note removed: "CAN1_RX"
- note removed: "CAN1_TX"
- note removed: "CAN\n"
- note removed: "DESCRIPTION:"
- note removed: "Fuses\n"
- note removed: "Inputs"
- note removed: "Outputs"
- note removed: "Outputs Control"
- note removed: "SPI1_MISO"
- note removed: "SPI1_MOSI\n"
- note removed: "SPI1_SCK"
- note removed: "STM CLOCK\n"
- note removed: "STM Power filtration"
- note removed: "STM RESET\n"
- note removed: "STM STATE"
- note removed: "STM\n"
- note removed: "STM_OK - green led\nSTM_FATAL_ERROR - red led\nSTM_SOFT_ERROR - yellow led\nSTM_??? - ??? led"
- note removed: "SWD"
- note removed: "SWDCLK\n"
- note removed: "SWDIO\n"
- note removed: "TIM2_CH3\n"
- note removed: "TM"
- note removed: "Use PCT polyfuse\n"
- note removed: "VIN = VDD"
- note removed: "gdzie?\n"
