File: hardware/SB-Spoko Bezpieczniki.kicad_pcb (KiCad board)
At the start: 4 copper layers, 179 x 60 mm, 143 parts, among them IC1 STM32L4P5RET6, J1 SWD, J2 Conn_02x20_Odd_Even, Q1 Q_NMOS_DGS, Q2 Q_NMOS_DGS, Q3 Q_NMOS_DGS, Q4 Q_NMOS_DGS, Q5 Q_NMOS_DGS, SW1 RESET, U1 AS222-35PN-933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

Commit message: Plz Janek powiedz mi ze jest ok
Routing:
- net V_PUMP: track 31.9 -> 55.0 mm
- net WHEEL: track 34.2 -> 37.3 mm
- net +24V: track 23.2 -> 26.0 mm, vias 12 -> 8
- net TSAL_LOGIC: track 19.3 -> 22.1 mm
- net WSS_RR: track 137.6 -> 134.9 mm
- net WSS_FR: track 145.6 -> 143.0 mm
- net USB_DP: track 114.5 -> 112.0 mm
- net USB_DM: track 119.2 -> 116.7 mm
- net V_SAFETY: track 47.5 -> 49.7 mm
- net WSS_FL: track 135.4 -> 133.3 mm
- net WSS_RL: track 126.8 -> 124.8 mm
- net MISO: track 128.7 -> 130.4 mm
- net TSAL_HV: track 19.8 -> 21.4 mm
- net SCK: track 131.3 -> 132.9 mm
- net USB_DEBUG_DM: track 112.9 -> 111.3 mm
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Other:
- board size 179 x 60 mm -> 166.4 x 60 mm

Commit message: added traceswo from pin 55 to progrmator
Connections:
- IC1 pad 55: LED_1_CONTROL -> SWO
- IC1 pad 57: unconnected-(IC1-Pad57) -> LED_1_CONTROL
- J1 pad 6: unconnected-(J1-Pad6) -> SWO
Routing:
- net SWO: track 0.00 -> 22.5 mm, vias 0 -> 1
- net LED_1_CONTROL: track 134.5 -> 140.4 mm

Commit message: preproduction bug fixes
Parts:
- removed C38, C39, C40: 100nF, Capacitor_SMD:C_0603_1608Metric
- Y1: value THE_CLOCK -> Crystal_GND24
- moved C25 1.03 mm to (106.2, 123.8), turned to 90 degrees
- moved C34 0.31 mm to (242.8, 87.5)
- moved Y1 0.22 mm to (239.8, 87.5), turned to 0 degrees
- moved C35 0.14 mm to (236.8, 87.4), turned to 90 degrees
- turned R32 to -90 degrees
Connections:
- Y1 pad 1: STM_CLK_IN -> STM_CKL_OUT
- Y1 pad 2: STM_CKL_OUT -> GND
- Y1 pad 3: (no net) -> STM_CLK_IN
- Y1 pad 4: (no net) -> GND
Routing:
- net V_PUMP: track 55.0 -> 42.6 mm
- net +5V: track 309.4 -> 318.2 mm, vias 9 -> 10
- net +3V3: track 419.3 -> 423.0 mm
- net STM_CKL_OUT: track 4.72 -> 6.52 mm
- net MONO_NTC: track 107.3 -> 108.9 mm
- net 3.3V_STM_POWER: track 65.9 -> 67.4 mm
- net GND: track 52.8 -> 53.5 mm, vias 35 -> 77
- net Net-(Q4-Pad2): track 4.07 -> 4.77 mm
- net WATER_P: track 107.3 -> 108.0 mm
