File: hardware/SB-Spoko Bezpieczniki.kicad_pcb (KiCad board)
At the start: 4 copper layers, 166.4 x 60 mm, 146 parts, among them IC1 STM32L4P5RET6, IC2 NCS20061MUTAG, IC3 NIS4461MT1TXG, IC4 NIS6351MT2TXG, J1 SWD, J2 Conn_02x20_Odd_Even, J3 M80-8420445, Q1 Q_NMOS_DGS, Q2 Q_NMOS_DGS, Q3 Q_NMOS_DGS, Q4 Q_NMOS_DGS, Q5 Q_NMOS_DGS, SW1 RESET, U1 AS222-35PN-933, U11 MCP2558FD-xSN, U12 SMART FUSE, U13 SMART FUSE, U14 SMART FUSE, U15 SMART FUSE, U16 FOD8802DR2, U17 FOD8802DR2, U2 LM2596S-12, U3 LM2596S-5, U4 LM317_SOT-223, U5 VOH1016AB-T2, U6 VOH1016AB-T2, U7 VOH1016AB-T2, U8 VOH1016AB-T2, U9 VOH1016AB-T2, Y1 Crystal_GND24_Small

Commit message: changed some footprints for clarity, and made some progress on board
Parts:
- removed C17, C19, C21, C23: 10nF, Capacitor_SMD:C_0603_1608Metric
- removed C18, C20, C22, C24: 100nF, Capacitor_SMD:C_0603_1608Metric
- removed U16, U17: FOD8802DR2, FOD8802DR2:SOIC127P600X175-8N
- removed U5, U6, U7, U8, U9: VOH1016AB-T2, Package_DIP:SMDIP-6_W7.62mm
- added D1: D_SCH, Diode_SMD:D_0603_1608Metric, F.Cu at (176.4, 57.4)
- added D11: D_SCH, Diode_SMD:D_0603_1608Metric, F.Cu at (195.7, 54.8)
- added D2: D_SCH, Diode_SMD:D_0603_1608Metric, F.Cu at (176.4, 54.8)
- added F3: Polyfuse, Fuse:Fuse_2010_5025Metric, F.Cu at (230.0, 105.4)
- added IC5: NIS4461MT1TXG, NIS4461MT1TXG:SON50P300X300X80-11N, F.Cu at (227.8, 105.4)
- added ILIM5: ?, Resistor_SMD:R_0603_1608Metric, F.Cu at (243.4, 30.0)
- added ILIM6: ?, Resistor_SMD:R_0603_1608Metric, F.Cu at (234.2, 19.6)
- added IMON2: 1k, Resistor_SMD:R_0603_1608Metric, F.Cu at (232.1, 23.8)
- added J4: M80-8661022, M80-8661022:M808661022, F.Cu at (187.0, 39.6)
- added O1: FOD8802DR2_IMG, FOD8802DR2:SOIC127P600X175-8N, F.Cu at (206.1, 146.5)
- added O2: FOD8802DR2_IMG, FOD8802DR2:SOIC127P600X175-8N, F.Cu at (235.9, 136.8)
- added O3: FOD8802DR2_IMG, FOD8802DR2:SOIC127P600X175-8N, F.Cu at (221.0, 136.8)
- added O4: FOD8802DR2_IMG, FOD8802DR2:SOIC127P600X175-8N, F.Cu at (206.1, 136.8)
- added O5: FOD8802DR2_IMG, FOD8802DR2:SOIC127P600X175-8N, F.Cu at (221.0, 146.5)
- added R45: --, Resistor_SMD:R_0603_1608Metric, F.Cu at (206.3, 38.6)
- added R46: --, Resistor_SMD:R_0603_1608Metric, F.Cu at (202.3, 43.7)
- added R48: 10k, Resistor_SMD:R_0603_1608Metric, F.Cu at (202.3, 41.2)
- added R49: 10k, Resistor_SMD:R_0603_1608Metric, F.Cu at (202.3, 38.6)
- added R5: --, Resistor_SMD:R_0603_1608Metric, F.Cu at (180.5, 54.7)
- added R50: 100, Resistor_SMD:R_0603_1608Metric, F.Cu at (277.8, 90.0)
- added R51: 100, Resistor_SMD:R_0603_1608Metric, F.Cu at (273.7, 95.9)
- added R52: 0, Resistor_SMD:R_0603_1608Metric, F.Cu at (273.7, 90.0)
- added R53: 10k, Resistor_SMD:R_0603_1608Metric, F.Cu at (226.8, 31.8)
- added R54: R_Small, Resistor_SMD:R_0603_1608Metric, F.Cu at (259.8, 51.6)
- added R6: --, Resistor_SMD:R_0603_1608Metric, F.Cu at (176.4, 59.9)
- C15, C31, C33, C36, C37, D12, D13, D14, D15, D16, R20, R21, R22, R23, R25, R26, R27, R28, R29, R3, R30, R31, R32, R33, R34, R35, R36: moved to F.Cu
- C16: value 100nF -> 0; moved to F.Cu
- C39: value C? -> 100nF
- IC2: value NCS20061MUTAG -> NCS20061MUTAG_IMG
- Q1, Q2, Q3, Q4, Q5: value Q_NMOS_DGS -> Q_NMOS_GSD; moved to F.Cu
- R10, R13, R14, R9: value 4k7 -> --; moved to F.Cu
- R11, R12, R15, R16, R7, R8: value 4k7 -> 10k; moved to F.Cu
- R17, R18, R41, R42: value R_Small -> 10k
- moved C15 105.6 mm to (238.2, 19.6), turned to 0 degrees
- moved R12 104.2 mm to (224.0, 153.0)
- moved R11 102.6 mm to (223.2, 155.6), turned to 180 degrees
- moved D14 99.3 mm to (221.4, 152.9)
- moved C16 88.5 mm to (232.1, 26.3), turned to 0 degrees
- moved R14 83.1 mm to (212.9, 152.9)
- moved R13 81.5 mm to (212.0, 155.7), turned to 180 degrees
- moved SW1 81.1 mm to (217.5, 78.9)
- moved D15 78.3 mm to (210.3, 152.9)
- moved Q2 68.0 mm to (192.2, 169.6), turned to -90 degrees
- moved R28 63.7 mm to (194.8, 169.6), turned to 90 degrees
- moved R30 63.2 mm to (192.2, 172.2), turned to 180 degrees
- moved R10 62.7 mm to (201.6, 152.9)
- moved R29 62.4 mm to (189.6, 169.6), turned to 90 degrees
- moved R9 61.2 mm to (200.8, 155.7), turned to 180 degrees
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Connections:
- net /Fusses/WATER/POT_FLAG renamed /Fusses/WATER-POTENTIOMMETER/WATER/POT_FLAG
- net CONVERT_5V renamed 5V_CONVERT_24V
- net TD renamed SPARE_2_SENSE
- C10 pad 1: 3.3V_STM_POWER -> GND
- C10 pad 2: GND -> 3.3V_STM_REF+
- C15 pad 1: Net-(C15-Pad1) -> /Fusses/Supply/IMON
- C16 pad 1: GND -> Net-(C16-Pad1)
- C16 pad 2: +3V3 -> GND
- C26 pad 1: BSPD/ESB_IMON -> BSPD/EBS_IMON
- C6 pad 1: V_PUMP -> PUMP_12V
- C8 pad 1: V_PUMP -> PUMP_12V
- D18 pad 1: CAR_CAN+ -> CAR_CAN-
- D18 pad 2: CAR_CAN- -> CAR_CAN+
- D3 pad 1: PUMP -> PUMP_24V
- D5 pad 1: PUMP -> PUMP_24V
- F1 pad 1: BSPD/ESB_24V -> BSPD/EBS_24V
- IC1 pad 13: 3.3V_STM_POWER -> 3.3V_STM_REF+
- IC1 pad 2: unconnected-(IC1-Pad2) -> SPARE_3_SENSE_SIG
- IC1 pad 24: unconnected-(IC1-Pad24) -> BSPD/EBS_STATE
- IC1 pad 25: unconnected-(IC1-Pad25) -> BSPD/EBS_IMON
- IC1 pad 26: N_AMS -> WATER/POT_IMON
- IC1 pad 27: N_SPARE -> WATER/POT_STATE
- IC1 pad 28: N_TSMS -> WATER/POT_ENABLE
- IC1 pad 29: BUZZER_CONTROL -> Net-(IC1-Pad29)
- IC1 pad 37: unconnected-(IC1-Pad37) -> DV_SENSE_SIG
- IC1 pad 38: unconnected-(IC1-Pad38) -> FIREWALL_SENSE_SIG
- IC1 pad 39: unconnected-(IC1-Pad39) -> HVD_SENSE_SIG
- IC1 pad 40: unconnected-(IC1-Pad40) -> HV_SENSE_SIG
- IC1 pad 44: CAN_RX -> Net-(IC1-Pad44)
- IC1 pad 45: CAN_TX -> Net-(IC1-Pad45)
- IC1 pad 51: unconnected-(IC1-Pad51) -> INVERTER_SENSE_SIG
- IC1 pad 52: unconnected-(IC1-Pad52) -> SPARE_1_SENSE_SIG
- IC1 pad 53: unconnected-(IC1-Pad53) -> SPARE_2_SENSE_SIG
- IC1 pad 56: N_TD -> unconnected-(IC1-Pad56)
- IC1 pad 58: N_HVD -> unconnected-(IC1-Pad58)
- IC1 pad 62: EN_MOSFET -> unconnected-(IC1-Pad62)
- IC3 pad 10: BSPD/ESB_24V -> BSPD/EBS_24V
- IC3 pad 5: BSPD/ESB_IMON -> BSPD/EBS_IMON
- IC3 pad 6: BSPD/ESB_24V -> BSPD/EBS_24V
- IC3 pad 7: BSPD/ESB_24V -> BSPD/EBS_24V
- IC3 pad 8: BSPD/ESB_24V -> BSPD/EBS_24V
- IC3 pad 9: BSPD/ESB_24V -> BSPD/EBS_24V
- IC4 pad 7: /Fusses/WATER/POT_EN -> /Fusses/WATER-POTENTIOMMETER/WATER/POT_EN
- ILIM1 pad 1: BSPD/ESB_24V -> BSPD/EBS_24V
- ILIM2 pad 1: BSPD/ESB_24V -> BSPD/EBS_24V
- IMON1 pad 1: BSPD/ESB_IMON -> BSPD/EBS_IMON
- J2 pad 30: USB_DP -> unconnected-(J2-Pad30)
- J2 pad 32: USB_DM -> unconnected-(J2-Pad32)
- J2 pad 5: RES_REF+ -> Net-(J2-Pad5)
- J2 pad 6: WATER_P -> WATER_1_PRESSURE
- J2 pad 7: RES_REF- -> GND
- JP1 pad 1: CAR_CAN- -> CAR_CAN+
- L1 pad 2: V_PUMP -> PUMP_12V
- L3 pad 1: PUMP -> PUMP_24V
- Q1 pad 2: Net-(Q1-Pad2) -> GND
- Q1 pad 3: GND -> Net-(Q1-Pad3)
- Q2 pad 2: Net-(Q2-Pad2) -> GND
- Q2 pad 3: GND -> Net-(Q2-Pad3)
- Q3 pad 2: Net-(Q3-Pad2) -> GND
- Q3 pad 3: GND -> Net-(Q3-Pad3)
- Q4 pad 2: Net-(Q4-Pad2) -> GND
- Q4 pad 3: GND -> Net-(Q4-Pad3)
- Q5 pad 2: Net-(Q5-Pad2) -> GND
- Q5 pad 3: GND -> Net-(Q5-Pad3)
- R10 pad 1: Net-(D13-Pad1) -> Net-(D12-Pad1)
- R10 pad 2: Net-(C17-Pad1) -> HV_SENSE
- R11 pad 1: Net-(C19-Pad1) -> GND
- R11 pad 2: AMS -> HVD_SENSE_SIG
- R12 pad 1: Net-(D14-Pad1) -> GND
- R12 pad 2: Net-(C19-Pad1) -> HV_SENSE_SIG
- R13 pad 1: Net-(C21-Pad1) -> Net-(D13-Pad1)
- R14 pad 1: Net-(D15-Pad1) -> Net-(D14-Pad1)
- R14 pad 2: Net-(C21-Pad1) -> SPARE_3_SENSE
- R15 pad 1: Net-(C23-Pad1) -> GND
- R15 pad 2: SPARE -> SPARE_2_SENSE_SIG
- R16 pad 1: Net-(D16-Pad1) -> GND
- R16 pad 2: Net-(C23-Pad1) -> SPARE_3_SENSE_SIG
- R19 pad 2: CAR_CAN+ -> CAR_CAN-
- R21 pad 1: BUZZER_CRL -> BUZZER_CONTROL
- R21 pad 2: Net-(Q1-Pad2) -> Net-(Q1-Pad1)
- R22 pad 1: Net-(Q1-Pad2) -> Net-(Q1-Pad1)
- R23 pad 2: Net-(Q1-Pad1) -> Net-(Q1-Pad3)
- R25 pad 1: LED_2_CRL -> LED_2_CONTROL
- R25 pad 2: Net-(Q2-Pad2) -> Net-(Q5-Pad1)
- R26 pad 1: Net-(Q2-Pad2) -> Net-(Q5-Pad1)
- R27 pad 2: Net-(Q2-Pad1) -> Net-(Q5-Pad3)
- R28 pad 1: LED_1_CRL -> LED_1_CONTROL
- R28 pad 2: Net-(Q3-Pad2) -> Net-(Q2-Pad1)
- R29 pad 1: Net-(Q3-Pad2) -> Net-(Q2-Pad1)
- R3 pad 1: +3V3 -> 3.3V_STM_POWER
- R30 pad 2: Net-(Q3-Pad1) -> Net-(Q2-Pad3)
- R31 pad 2: Net-(Q4-Pad2) -> Net-(Q4-Pad1)
- R32 pad 1: Net-(Q4-Pad2) -> Net-(Q4-Pad1)
- R33 pad 2: Net-(Q4-Pad1) -> Net-(Q4-Pad3)
- R34 pad 2: Net-(Q5-Pad2) -> Net-(Q3-Pad1)
- R35 pad 1: Net-(Q5-Pad2) -> Net-(Q3-Pad1)
- R36 pad 2: Net-(Q5-Pad1) -> Net-(Q3-Pad3)
- R41 pad 1: GND -> Net-(O4-Pad8)
- R41 pad 2: WATER/POT_STATE -> +3V3
- R42 pad 2: /Fusses/WATER/POT_EN -> WATER/POT_STATE
- R43 pad 1: BSPD/ESB_STATE -> BSPD/EBS_STATE
- R7 pad 1: Net-(C15-Pad1) -> GND
- R7 pad 2: TSMS -> INVERTER_SENSE_SIG
- R8 pad 1: Net-(D12-Pad1) -> GND
- R8 pad 2: Net-(C15-Pad1) -> SPARE_1_SENSE_SIG
- R9 pad 1: Net-(C17-Pad1) -> Net-(D11-Pad1)
- R9 pad 2: HVD -> HVD_SENSE
- U1 pad 45: unconnected-(U1-Pad45) -> SPARE_1_24V
- U11 pad 6: CAR_CAN+ -> CAR_CAN-
- U11 pad 7: CAR_CAN- -> CAR_CAN+
- U13 pad 21: WHEEL_SPEED_1_24V -> ODRIVE_24V
- U13 pad 22: WHEEL_SPEED_1_24V -> ODRIVE_24V
- U13 pad 25: DASH_24V -> FAN_R_24V
- U13 pad 26: DASH_24V -> FAN_R_24V
- U13 pad 27: LAPTIMER_24V -> FAN_L_24V
- U13 pad 28: LAPTIMER_24V -> FAN_L_24V
- U13 pad 29: FAN_L_24V -> LAPTIMER_24V
- U13 pad 3: ODRIVE_24V -> WHEEL_SPEED_1_24V
- U13 pad 30: FAN_L_24V -> LAPTIMER_24V
- U13 pad 31: FAN_R_24V -> DASH_24V
- U13 pad 32: FAN_R_24V -> DASH_24V
- U13 pad 4: ODRIVE_24V -> WHEEL_SPEED_1_24V
- U14 pad 27: /Fusses/Fuse 2/VOUT_3 -> WHEEL_SPEED_2_24V
- U14 pad 28: /Fusses/Fuse 2/VOUT_3 -> WHEEL_SPEED_2_24V
- U14 pad 29: WHEEL_SPEED_2_24V -> LIDAR_24V
- U14 pad 3: ASMS_24V -> SPARE_1_24V
- U14 pad 30: WHEEL_SPEED_2_24V -> LIDAR_24V
- U14 pad 31: LIDAR_24V -> ASMS_24V
- U14 pad 32: LIDAR_24V -> ASMS_24V
- U14 pad 4: ASMS_24V -> SPARE_1_24V
- U2 pad 4: V_PUMP -> PUMP_12V
Routing:
- net +3V3: track 414.1 -> 87.0 mm, vias 7 -> 2
- net N_AMS: track 169.7 -> 0.00 mm, vias 2 -> 0
- net EN_MOSFET: track 157.3 -> 0.00 mm, vias 3 -> 0
- net N_TD: track 151.3 -> 0.00 mm, vias 2 -> 0
- net BUZZER_CONTROL: track 142.7 -> 0.00 mm, vias 2 -> 0
- net N_HVD: track 139.5 -> 0.00 mm, vias 2 -> 0
- net Net-(IC1-Pad29): track 0.00 -> 123.8 mm, vias 0 -> 1
- net Net-(R20-Pad1): track 116.1 -> 0.00 mm, vias 2 -> 1
- net +5V: track 299.1 -> 186.6 mm, vias 10 -> 2
- net WATER/POT_IMON: track 0.00 -> 110.0 mm, vias 0 -> 1
- net unconnected-(IC1-Pad62): track 0.00 -> 104.3 mm, vias 0 -> 1
- net BREAK_LIGHT_GATE: track 101.2 -> 1.90 mm, vias 1 -> 0
- net RTDS_GATE: track 98.8 -> 0.00 mm, vias 1 -> 0
- net AMS: track 93.3 -> 0.00 mm
- net unconnected-(U1-Pad27): track 102.2 -> 15.4 mm, vias 1 -> 0
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- added copper zone on F.Cu, net 5V_CONVERT_24V
- removed copper zone on F.Cu, net Net-(C3-Pad1)
Other:
- board text removed: "3.3v"
- board text removed: "ERROR"
- board text removed: "OK"
- board text removed: "WARNING 1"
- board text removed: "WARNING 2"
- board text removed: "gnd"
- board text removed: "n_rst"
- board text removed: "swclk"
- board text removed: "swdio"
