File: hardware/eFuse 24V.kicad_sch (KiCad schematic)
At the start: 9 parts, among them IC2 NCS20061MUTAG, IC3 NIS4461MT1TXG

Commit message: changed some footprints for clarity, and made some progress on board
Parts:
- removed IC2: NCS20061MUTAG, NCS20061MUTAG:SON50P160X160X55-7N, symbol NCS20061MUTAG:NCS20061MUTAG
- added IC2: NCS20061MUTAG_IMG, NCS20061MUTAG:SON50P160X160X55-7N, symbol NCS20061MUTAG:NCS20061MUTAG_IMG
Connections:
- net +3V3: now also IC2.5 (V+)
- net EN/FAULT: now also IC2.4
- net GND: now also IC2.1 (-V)
- net at R43.2: now also IC2.3, IC2.6
- no-connect marks 0 -> 1
Other:
- moved on the sheet: R43
