File: hardware/Smart fuse.kicad_sch (KiCad schematic)
At the start: 2 parts, among them U12 SMART FUSE

Commit message: debuged the board, changed one opto for mosfet, changed the way water and potentiometers were supplied. Also standrised opamps (yoinked opamps from data Data_Acquisition_Cards)
Parts:
- renumbered C1 to C32, U12 to U15
Changed lines of the file:
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@@
   (symbol (lib_id "Device:C") (at 156.21 68.58 270)
     (in_bom yes) (on_board yes)
-    (property "Reference" "C1" (id 0) (at 156.21 62.1792 90))
+    (property "Reference" "C32" (id 0) (at 156.21 62.1792 90))
     (property "Value" "100nF" (id 1) (at 156.21 64.4906 90))
     (property "Footprint" "Capacitor_SMD:C_0603_1608Metric" (id 2) (at 152.4 69.5452 0)
@@
   (symbol (lib_id "VN9D30Q100F:VN9D30Q100F") (at 144.78 76.2 0)
     (in_bom yes) (on_board yes)
-    (property "Reference" "U12" (id 0) (at 132.08 71.12 0))
+    (property "Reference" "U15" (id 0) (at 132.08 71.12 0))
     (property "Value" "SMART FUSE" (id 1) (at 132.08 73.66 0))
     (property "Footprint" "VN9D30Q100F:QFN-32_EP_6x6_Pitch0.5mm" (id 2) (at 154.94 72.39 0)
