File: hardware/eFuse supply 24V.kicad_sch (KiCad schematic)
At the start: 7 parts, among them IC5 NIS4461MT1TXG

Commit message: finished new wersion of the board
Connections:
- net EN/FAULT: no longer names the net of IC5.3 (EN/FLT)
- no-connect marks 0 -> 1
Changed lines of the file:
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@@
   (junction (at 168.91 89.535) (diameter 0) (color 0 0 0 0)
   )
+  (no_connect (at 128.27 84.455))
   (wire (pts (xy 114.935 99.695) (xy 121.285 99.695))
     (stroke (width 0) (type default) (color 0 0 0 0))
@@
     (stroke (width 0) (type default) (color 0 0 0 0))
   )
-  (wire (pts (xy 108.585 84.455) (xy 130.81 84.455))
+  (wire (pts (xy 128.27 84.455) (xy 130.81 84.455))
     (stroke (width 0) (type default) (color 0 0 0 0))
   )
@@
     (effects (font (size 3 3) bold) (justify left bottom))
   )
-  (label "EN{slash}FAULT" (at 108.585 84.455 180)
-    (effects (font (size 1.27 1.27)) (justify right bottom))
-  )
   (hierarchical_label "VOUT" (shape output) (at 171.45 107.95 0)
     (effects (font (size 1.27 1.27)) (justify left))
@@
     (effects (font (size 1.27 1.27)) (justify right))
   )
-  (symbol (lib_id "NIS4461MT1TXG:NIS4461MT1TXG") (at 130.81 79.375 0) (unit 1)
+  (symbol (lib_id "NIS4461MT1TXG:NIS4461MT1TXG") (at 130.81 79.375 0)
     (in_bom yes) (on_board yes) (fields_autoplaced)
     (property "Reference" "IC5" (id 0) (at 148.59 71.12 0))
@@
     (pin "9")
   )
-  (symbol (lib_id "Device:R_Small") (at 160.655 119.38 270) (unit 1)
+  (symbol (lib_id "Device:R_Small") (at 160.655 119.38 270)
     (in_bom yes) (on_board yes)
     (property "Reference" "ILIM6" (id 0) (at 160.655 121.92 90))
@@
     (pin "2")
   )
-  (symbol (lib_id "Device:R_Small") (at 112.395 94.615 0) (unit 1)
+  (symbol (lib_id "Device:R_Small") (at 112.395 94.615 0)
     (in_bom yes) (on_board yes)
     (property "Reference" "IMON2" (id 0) (at 105.41 93.345 0)
@@
     (pin "2")
   )
-  (symbol (lib_id "power:GND") (at 114.935 111.76 0) (unit 1)
+  (symbol (lib_id "power:GND") (at 114.935 111.76 0)
     (in_bom yes) (on_board yes) (fields_autoplaced)
     (property "Reference" "#PWR0150" (id 0) (at 114.935 118.11 0)
@@
     (pin "1")
   )
-  (symbol (lib_id "Device:Polyfuse") (at 161.29 107.95 270) (unit 1)
+  (symbol (lib_id "Device:Polyfuse") (at 161.29 107.95 270)
     (in_bom yes) (on_board yes)
     (property "Reference" "F3" (id 0) (at 161.29 105.41 90))
@@
     (pin "2")
   )
-  (symbol (lib_id "Device:C_Small") (at 102.235 94.615 0) (unit 1)
+  (symbol (lib_id "Device:C_Small") (at 102.235 94.615 0)
     (in_bom yes) (on_board yes)
     (property "Reference" "C15" (id 0) (at 96.52 93.345 0)
@@
     (pin "2")
   )
-  (symbol (lib_id "Device:C_Small") (at 121.285 94.615 0) (unit 1)
+  (symbol (lib_id "Device:C_Small") (at 121.285 94.615 0)
     (in_bom yes) (on_board yes)
     (property "Reference" "C16" (id 0) (at 116.205 93.345 0)
@@
     (pin "2")
   )
-  (symbol (lib_id "Device:R_Small") (at 160.655 111.76 270) (unit 1)
+  (symbol (lib_id "Device:R_Small") (at 160.655 111.76 270)
     (in_bom yes) (on_board yes)
     (property "Reference" "ILIM5" (id 0) (at 160.655 114.3 90))
